File: S0001-Strand-Burner-DAQ/src/S0001-Strand-Burner-DAQ/S0001-Strand-Burner-DAQ.kicad_sch (KiCad schematic)
At the start: 20 parts

Commit message: Updated Schematic
Parts:
- removed BT? (x2): Battery, symbol S0001-Strand-Burner-DAQ:Battery
- removed D?: Diode, Diode_SMD:D_SOD-523, symbol S0001-Strand-Burner-DAQ:Diode
- removed H? (x4): Mounting-Hole, symbol S0001-Strand-Burner-DAQ:Mounting-Hole
- removed L?: INDUCTOR, symbol S0001-Strand-Burner-DAQ:INDUCTOR
- removed Q?: Transistor, Package_TO_SOT_THT:TO-92_Inline, symbol S0001-Strand-Burner-DAQ:Transistor
- removed R?: R_US, symbol S0001-Strand-Burner-DAQ:R_US
- removed SW?: SW_DIP_x01, symbol S0001-Strand-Burner-DAQ:SW_DIP_x01
- added H? (x4): Mounting-Hole, symbol S0001-Strand-Burner-DAQ:Mounting-Hole
- added J?: Solenoid_Connector, CONN_140-502-417-011_EDA, symbol S0001-Strand-Burner-DAQ:Solenoid_Connector
- added Q? (x2): MOSFET, Package_TO_SOT_SMD:LFPAK33, symbol S0001-Strand-Burner-DAQ:MOSFET
- added R?: R_US, symbol S0001-Strand-Burner-DAQ:R_US
Connections:
- net Earth: no longer D?.1 (K), J?.1
- net Start: now reaches A?.13 (D10)
- net Start: now also Q?.4 (G), Q?.4 (G)
- net SOLENOID DRIVER: now reaches R?.1
- net SOLENOID DRIVER: now also D?.1 (K), J?.1, J?.2, Q?.5 (D), R?.2
- net CarBat renamed 12V
- net 12V: now also Q?.1 (S), Q?.1 (S), Q?.2 (S), Q?.2 (S), Q?.3 (S), Q?.3 (S)
- net Load Cell Power renamed 5V
- net PWM-5 renamed Strand-2
- net Strand-2: now also A?.9 (D6), R?.2
- removed net PWM-6: A?.9 (D6), J?.4, R?.2
- new net: J?.1, Q?.5 (D), R?.1
- new net Strand-3: J?.4
Other:
- note added: "NOTES: CHANGE BATTERIES TO DIFFERENT CONNECTORS TO POWER CHANGE SOLENOID TO TRANSISTOR + POWER SUPPLY UPDATE FOOTPRINT W/ CONNECTOR"
- note added: "Solenoid Driver"
- note added: "connector here"
- note removed: "Load Cell Connector Pressure Connector What to input for the SD module"
- note removed: "NEED TO KNOW:"
- moved on the sheet: D?, LOGO?, R?
